File: TBX01.brd (EAGLE design)
At the start: 49.8 x 40.1 mm, 75 parts, among them IC1 TPS62120, SW1 SW-TACTILE-PTS840P, SW2 SW-TACTILE-PTS840P, SW3 SW-TACTILE-PTS840P, SW4 SW-TACTILE-PTS840P, U3 STM32L151CCT6, U6 MCP73833, X2 FH12-10S-0.5SH, Y1 CRYSTAL.ABS07

Commit message: TBX01 v0.2
Parts:
- removed C13: 10uF, microbuilder:0603
- added D1: (no value), microbuilder:SMADIODE
Connections:
- new net N$54: C5.2, D1.A, JTAG1.15, S1.1, U3.7
- net GND: no longer C13.2
- net N$10: now also D1.C; no longer C5.2, JTAG1.15, S1.1, U3.7
- net VDD: no longer C13.1
Changed lines of the file:
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@@
 <element name="C11" library="microbuilder" package="0603" value="100nF" x="72.39" y="59.944"/>
 <element name="C12" library="microbuilder" package="0603" value="100nF" x="72.39" y="58.166"/>
-<element name="C13" library="microbuilder" package="0603" value="10uF" x="72.39" y="56.388"/>
 <element name="C14" library="microbuilder" package="0603" value="1uF" x="23.7236" y="12.446" rot="R180"/>
 <element name="C15" library="microbuilder" package="0603" value="1uF" x="20.0406" y="12.446" rot="R180"/>
@@
 <element name="R22" library="microbuilder" package="0603" value="4.7k" x="63.754" y="41.91"/>
 <element name="R23" library="microbuilder" package="0603" value="4.7k" x="63.754" y="40.132"/>
+<element name="D1" library="microbuilder" package="SMADIODE" value="" x="-2.5908" y="-8.636"/>
 </elements>
 <signals>
@@
 <contactref element="C10" pad="2"/>
 <contactref element="C11" pad="2"/>
-<contactref element="C13" pad="2"/>
 <contactref element="X2" pad="10"/>
 <contactref element="X2" pad="9"/>
@@
 <wire x1="20.792" y1="10.414" x2="20.8138" y2="10.414" width="0.3048" layer="1"/>
 <wire x1="20.8138" y1="10.414" x2="20.815" y2="10.4128" width="0.3048" layer="1"/>
+<wire x1="28.4344" y1="8.4582" x2="28.614" y2="8.6378" width="0.3048" layer="16"/>
+<wire x1="28.614" y1="8.6378" x2="28.614" y2="10.414" width="0.3048" layer="16"/>
 <wire x1="73.24" y1="68.834" x2="71.54" y2="70.612" width="0" layer="19" extent="1-1"/>
 <wire x1="73.24" y1="67.056" x2="73.24" y2="68.834" width="0" layer="19" extent="1-1"/>
@@
 <wire x1="73.24" y1="59.944" x2="73.24" y2="61.722" width="0" layer="19" extent="1-1"/>
 <wire x1="73.24" y1="58.166" x2="73.24" y2="59.944" width="0" layer="19" extent="1-1"/>
-<wire x1="73.24" y1="56.388" x2="73.24" y2="58.166" width="0" layer="19" extent="1-1"/>
 <wire x1="64.604" y1="67.056" x2="71.54" y2="65.278" width="0" layer="19" extent="1-1"/>
-<wire x1="71.54" y1="49.276" x2="73.24" y2="56.388" width="0" layer="19" extent="1-1"/>
+<wire x1="71.54" y1="49.276" x2="73.24" y2="58.166" width="0" layer="19" extent="1-1"/>
 <wire x1="71.54" y1="47.498" x2="71.54" y2="49.276" width="0" layer="19" extent="1-1"/>
 <wire x1="71.54" y1="45.72" x2="71.54" y2="47.498" width="0" layer="19" extent="1-1"/>
@@
 <wire x1="3.132" y1="46.698" x2="1.73" y2="27.56" width="0" layer="19" extent="1-1"/>
 <wire x1="0.932" y1="48.298" x2="3.132" y2="46.698" width="0" layer="19" extent="1-1"/>
-<wire x1="28.4344" y1="8.4582" x2="28.614" y2="8.6378" width="0.3048" layer="16"/>
-<wire x1="28.614" y1="8.6378" x2="28.614" y2="10.414" width="0.3048" layer="16"/>
 </signal>
 <signal name="VDD">
@@
 <contactref element="C12" pad="1"/>
 <contactref element="C10" pad="1"/>
-<contactref element="C13" pad="1"/>
 <contactref element="X2" pad="7"/>
 <contactref element="X2" pad="6"/>
@@
 <wire x1="30.314" y1="1.524" x2="30.314" y2="4.826" width="0.4064" layer="16"/>
 <wire x1="30.314" y1="4.826" x2="30.314" y2="10.414" width="0.4064" layer="16"/>
+<wire x1="29.298" y1="4.826" x2="30.314" y2="4.826" width="0.4064" layer="16"/>
 <wire x1="71.54" y1="59.944" x2="71.54" y2="61.722" width="0" layer="19" extent="1-1"/>
 <wire x1="71.54" y1="58.166" x2="71.54" y2="59.944" width="0" layer="19" extent="1-1"/>
-<wire x1="71.54" y1="56.388" x2="71.54" y2="58.166" width="0" layer="19" extent="1-1"/>
-<wire x1="64.604" y1="47.244" x2="71.54" y2="56.388" width="0" layer="19" extent="1-1"/>
+<wire x1="64.604" y1="47.244" x2="71.54" y2="58.166" width="0" layer="19" extent="1-1"/>
 <wire x1="64.604" y1="45.466" x2="64.604" y2="47.244" width="0" layer="19" extent="1-1"/>
 <wire x1="64.604" y1="43.688" x2="64.604" y2="45.466" width="0" layer="19" extent="1-1"/>
@@
 <wire x1="21.082" y1="16.3576" x2="18.284" y2="13.3604" width="0" layer="19" extent="1-1"/>
 <wire x1="15.5956" y1="24.7904" x2="14.1224" y2="19.3294" width="0" layer="19" extent="1-1"/>
-<wire x1="29.298" y1="4.826" x2="30.314" y2="4.826" width="0.4064" layer="16"/>
 </signal>
 <signal name="TP">
@@
 <contactref element="U1" pad="19"/>
 <contactref element="U3" pad="46"/>
-<contactref element="C5" pad="2"/>
-<contactref element="U3" pad="7"/>
-<contactref element="S1" pad="1"/>
 <contactref element="S2" pad="1"/>
-<contactref element="JTAG1" pad="15"/>
 <contactref element="C19" pad="2"/>
-<wire x1="73.24" y1="45.72" x2="73.24" y2="70.612" width="0" layer="19" extent="1-1"/>
+<contactref element="D1" pad="C"/>
 <wire x1="48.09" y1="14.456" x2="73.24" y2="45.72" width="0" layer="19" extent="1-16"/>
-<wire x1="48.09" y1="7.344" x2="48.09" y2="14.456" width="0" layer="19" extent="16-16"/>
-<wire x1="40.386" y1="10.16" x2="48.09" y2="7.344" width="0" layer="19" extent="16-16"/>
-<wire x1="23.154" y1="26.174" x2="40.386" y2="10.16" width="0" layer="19" extent="16-16"/>
+<wire x1="23.154" y1="26.174" x2="48.09" y2="14.456" width="0" layer="19" extent="16-16"/>
 <wire x1="16.5862" y1="24.7904" x2="23.154" y2="26.174" width="0" layer="19" extent="1-16"/>
-<wire x1="14.1224" y1="20.32" x2="16.5862" y2="24.7904" width="0" layer="19" extent="1-1"/>
+<wire x1="-4.9403" y1="-8.636" x2="16.5862" y2="24.7904" width="0" layer="19" extent="1-1"/>
 </signal>
 <signal name="N$37">
@@
 <wire x1="24.904" y1="29.424" x2="73.24" y2="33.274" width="0" layer="19" extent="1-16"/>
 </signal>
+<signal name="N$54">
+<contactref element="U3" pad="7"/>
+<contactref element="S1" pad="1"/>
+<contactref element="D1" pad="A"/>
+<contactref element="JTAG1" pad="15"/>
+<contactref element="C5" pad="2"/>
+<wire x1="48.09" y1="7.344" x2="73.24" y2="70.612" width="0" layer="19" extent="1-16"/>
+<wire x1="40.386" y1="10.16" x2="48.09" y2="7.344" width="0" layer="19" extent="16-16"/>
+<wire x1="14.1224" y1="20.32" x2="40.386" y2="10.16" width="0" layer="19" extent="1-1"/>
+<wire x1="-0.2413" y1="-8.636" x2="14.1224" y2="20.32" width="0" layer="19" extent="1-1"/>
+</signal>
 </signals>

Commit message: TBX01 v0.2-r201508171545
On branch master
	.~lock.TBX-01_power.ods#
nothing added to commit but untracked files present (use "git add" to track)
Parts:
- D1: device microbuilder:SMADIODE -> microbuilder:SOD-123
- moved C7 75.3 mm to (8.00, 28.1), turned to 90 degrees
- moved C6 74.1 mm to (10.5, 28.1), turned to 90 degrees
- moved R14 65.7 mm to (6.25, 24.5), turned to 270 degrees
- moved C26 64.2 mm to (8.20, 35.5), flipped to the bottom
- moved C27 58.8 mm to (13.7, 35.5), flipped to the bottom
- moved D1 43.3 mm to (4.50, 34.1)
- moved Y1 22.4 mm to (9.25, 25.3)
- moved X1 18.4 mm to (11.9, 31.9), flipped to the bottom
- moved R10 3.47 mm to (42.5, 6.53), turned to 90 degrees
Connections:
- net N$18: now also Y1.2; no longer Y1.1
- net N$22: now also Y1.1; no longer Y1.2
Routing:
- net GND: track 125.9 -> 213.2 mm, vias 3 -> 7
- net N$54: track 0.00 -> 40.3 mm, vias 0 -> 2
- net VDD: track 87.2 -> 105.0 mm
- net N$21: track 0.00 -> 9.67 mm
- net N$18: track 0.00 -> 8.52 mm
- net N$28: track 0.00 -> 6.49 mm
- net N$27: track 0.00 -> 6.48 mm
- net D+: track 4.13 -> 0.00 mm
- net N$22: track 0.00 -> 3.66 mm
- net N$6: track 41.5 -> 42.3 mm
- net VIN: track 15.0 -> 14.3 mm

Commit message: TBX01 v0.2-r201508171633
Parts:
- moved C11 65.7 mm to (15.3, 27.5)
- moved C12 64.2 mm to (23.6, 16.4)
- moved C10 63.2 mm to (25.9, 18.8)
Routing:
- net N$25: track 0.00 -> 35.9 mm
- net DCDC-PWRGOOD: track 10.2 -> 32.4 mm, vias 1 -> 3
- net N$24: track 3.84 -> 17.1 mm
- net N$26: track 0.00 -> 6.91 mm, vias 0 -> 2
- net GND: track 213.2 -> 217.4 mm, vias 7 -> 8
- net VDD: track 105.0 -> 108.2 mm
- net N$54: track 40.3 -> 40.8 mm

Commit message: TBX01 v0.2-r201508172343
Parts:
- moved C10 5.78 mm to (23.9, 24.3)
- moved U1 2.68 mm to (26.6, 29.4)
- moved C12 2.39 mm to (21.7, 14.9)
- moved C11 2.19 mm to (14.1, 25.6), turned to 90 degrees
Connections:
- net GND: now also C11.1, C12.1; no longer C11.2, C12.2
- net VDD: now also C11.2, C12.2; no longer C11.1, C12.1
Routing:
- net N$48: track 5.89 -> 0.00 mm
- net N$46: track 5.38 -> 0.00 mm
- net N$45: track 4.84 -> 0.00 mm
- net GND: track 217.4 -> 213.3 mm
- net N$47: track 2.85 -> 0.00 mm
- net VDD: track 108.2 -> 111.0 mm
- net N$13: track 0.27 -> 2.92 mm
- net N$12: track 0.00 -> 2.23 mm

Commit message: TBX01 v0.2-r201508181539
Parts:
- moved C8 54.3 mm to (32.8, 28.1), flipped to the bottom
- moved C9 51.7 mm to (32.8, 30.3), flipped to the bottom
- moved R16 46.5 mm to (33.6, 17.1), flipped to the bottom, turned to 90 degrees
- moved R8 42.4 mm to (46.8, 28.1), flipped to the bottom, turned to 180 degrees
- moved R15 38.0 mm to (46.9, 20.3), flipped to the bottom, turned to 180 degrees
- moved R17 31.5 mm to (46.8, 24.3), flipped to the bottom, turned to 180 degrees
- moved R13 27.0 mm to (48.2, 35.8), turned to 270 degrees
- moved U1 3.56 mm to (26.6, 25.9)
- moved C14 2.78 mm to (24.5, 9.78)
- moved C12 2.21 mm to (23.3, 16.5)
- moved R9 1.83 mm to (42.5, 11.0), turned to 90 degrees
- moved LED1 1.73 mm to (46.9, 29.9)
- moved LED2 0.61 mm to (47.0, 26.0)
- moved LED3 0.48 mm to (47.0, 22.1)
- moved C15 0.37 mm to (20.1, 12.1)
Connections:
- net GND: now also C12.2; no longer C12.1
- net VDD: now also C12.1; no longer C12.2
Routing:
- net N$30: track 0.00 -> 26.0 mm, vias 0 -> 1
- net D-: track 3.31 -> 24.3 mm, vias 0 -> 3
- net D+: track 0.00 -> 20.7 mm, vias 0 -> 3
- net N$31: track 0.00 -> 19.3 mm, vias 0 -> 1
- net N$29: track 0.00 -> 17.9 mm, vias 0 -> 1
- net GND: track 213.3 -> 230.5 mm, vias 8 -> 9
- net N$17: track 0.00 -> 14.6 mm
- net N$23: track 0.00 -> 13.9 mm, vias 0 -> 2
- net N$39: track 0.00 -> 13.2 mm
- net N$33: track 0.00 -> 12.3 mm, vias 0 -> 1
- net N$32: track 0.00 -> 12.2 mm, vias 0 -> 1
- net N$34: track 0.00 -> 9.82 mm, vias 0 -> 1
- net N$35: track 0.00 -> 8.04 mm, vias 0 -> 1
- net N$11: track 0.00 -> 7.46 mm
- net N$54: track 40.8 -> 34.8 mm
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
Commit message: TBX01 v0.2-r201508181630
Routing:
- net GND: track 230.5 -> 231.7 mm
Changed lines of the file:
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@@
 <wire x1="1.25" y1="5.918" x2="4.826" y2="4.992" width="0" layer="19" extent="1-16"/>
 <wire x1="1.73" y1="27.56" x2="4.953" y2="30.353" width="0" layer="19" extent="1-1"/>
-<wire x1="29.0684" y1="24.1326" x2="24.726" y2="24.257" width="0" layer="19" extent="1-16"/>
 <wire x1="33.322" y1="9.718" x2="37.846" y2="10.16" width="0" layer="19" extent="1-1"/>
 <wire x1="33.6414" y1="28.067" x2="37.846" y2="25.4" width="0" layer="19" extent="16-16"/>
@@
 <wire x1="1.576" y1="14.334" x2="4.226" y2="19.634" width="0" layer="19" extent="16-16"/>
 <wire x1="44.1198" y1="8.5734" x2="45.89" y2="10.944" width="0" layer="19" extent="1-16"/>
+<wire x1="29.0684" y1="24.1326" x2="30.1472" y2="24.1326" width="0.3048" layer="16"/>
+<wire x1="30.1472" y1="24.1326" x2="30.2768" y2="24.003" width="0.3048" layer="16"/>
+<wire x1="30.2768" y1="24.003" x2="27.8184" y2="28.3826" width="0" layer="19" extent="1-16"/>
 </signal>
 <signal name="VDD">

Commit message: TBX01 v0.2-r201508190105
Parts:
- moved C26 11.3 mm to (17.9, 29.6), turned to 180 degrees
- moved C27 9.11 mm to (17.9, 27.4)
- moved C9 4.35 mm to (28.4, 30.6)
- moved X1 4.24 mm to (14.4, 28.5), turned to 270 degrees
- moved D1 3.51 mm to (7.16, 31.8), turned to 180 degrees
- moved R14 3.17 mm to (8.18, 21.9), turned to 0 degrees
- moved B1 2.72 mm to (22.4, 30.7)
- moved SW2 1.50 mm to (2.61, 28.0)
- moved C6 1.35 mm to (10.4, 26.7)
- moved C7 1.35 mm to (7.87, 26.7)
- moved Y1 1.35 mm to (9.12, 24.0)
- moved C8 1.12 mm to (31.8, 27.6), turned to 90 degrees
Routing:
- net N$5: track 23.0 -> 0.00 mm
- net N$36: track 2.22 -> 14.6 mm
- net BAT-STAT1: track 0.00 -> 10.4 mm, vias 0 -> 1
- net GND: track 231.7 -> 223.0 mm
- net N$53: track 0.00 -> 8.13 mm
- net N$51: track 0.00 -> 5.55 mm
- net BAT-PWRGOOD: track 0.00 -> 4.79 mm, vias 0 -> 1
- net N$21: track 9.67 -> 5.15 mm
- net VBAT: track 36.0 -> 40.2 mm
- net N$50: track 0.00 -> 1.86 mm
- net N$18: track 8.52 -> 7.23 mm
- net D-: track 24.3 -> 23.4 mm
- net D+: track 20.7 -> 21.5 mm
- net N$22: track 3.66 -> 4.28 mm

Commit message: TBX01 v0.2-r201508191318
Before nRF8001 move left
Parts:
- moved B1 2.54 mm to (22.4, 28.1)
- turned X1 to 90 degrees
Routing:
- net N$53: track 8.13 -> 1.28 mm
- net GND: track 223.0 -> 229.3 mm, vias 9 -> 10
- net N$51: track 5.55 -> 0.00 mm
- net N$48: track 0.00 -> 3.47 mm
- net N$46: track 0.00 -> 3.04 mm
- net N$45: track 0.00 -> 2.53 mm
- net N$50: track 1.86 -> 0.00 mm
