File: TBX01.brd (EAGLE design)
At the start: 49.8 x 40.1 mm, 75 parts, among them IC1 TPS62120, SW1 SW-TACTILE-PTS840P, SW2 SW-TACTILE-PTS840P, SW3 SW-TACTILE-PTS840P, SW4 SW-TACTILE-PTS840P, U3 STM32L151CCT6, U6 MCP73833, X2 FH12-10S-0.5SH, Y1 CRYSTAL.ABS07

Commit message: TBX01 v0.2-r201508201349
Parts:
- moved C20 77.1 mm to (2.11, 12.1)
- moved C18 74.0 mm to (3.43, 20.7), turned to 90 degrees
- moved R19 53.1 mm to (13.2, 31.0)
- moved C22 47.3 mm to (44.8, 1.98), turned to 90 degrees
- moved R20 42.9 mm to (27.5, 22.6)
- moved R21 37.5 mm to (34.6, 20.1)
- moved R12 37.4 mm to (36.6, 34.0), turned to 180 degrees
- moved R22 37.4 mm to (34.6, 18.5)
- moved R23 37.3 mm to (34.6, 16.8)
- moved C21 30.1 mm to (44.4, 31.2), turned to 90 degrees
- moved X1 18.4 mm to (32.8, 29.9), turned to 270 degrees
- moved R13 16.6 mm to (31.9, 32.7), turned to 180 degrees
- moved SW1 15.3 mm to (47.7, 36.2)
- moved SW4 15.3 mm to (47.2, 3.47)
- moved C26 11.6 mm to (29.4, 31.2), turned to 0 degrees
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Routing:
- net N$17: track 14.6 -> 60.1 mm, vias 0 -> 2
- net N$43: track 0.00 -> 35.6 mm, vias 0 -> 1
- net N$5: track 0.00 -> 28.5 mm
- net N$16: track 0.00 -> 24.4 mm
- net N$23: track 13.9 -> 36.2 mm, vias 2 -> 3
- net VDD: track 113.3 -> 127.9 mm, vias 2 -> 3
- net N$36: track 14.6 -> 2.29 mm
- net N$15: track 0.00 -> 10.7 mm
- net N$9: track 31.0 -> 37.2 mm
- net N$6: track 42.3 -> 48.4 mm
- net N$33: track 12.3 -> 18.4 mm
- net N$25: track 35.4 -> 29.6 mm, vias 0 -> 2
- net N$20: track 0.00 -> 5.69 mm
- net N$39: track 13.2 -> 7.72 mm
- net N$7: track 23.6 -> 29.0 mm
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Other:
- outline, holes or cut-outs redrawn

Commit message: TBX01 v0.2-r201508201530
Parts:
- moved C17 52.7 mm to (23.4, 29.8), flipped to the bottom
- moved R18 19.7 mm to (58.9, 30.0), flipped to the bottom
- moved B1 3.22 mm to (19.8, 30.0)
- moved JP4 0.38 mm to (39.5, 38.2)
- moved JP3 0.20 mm to (39.5, 35.9)
Routing:
- net N$36: track 2.29 -> 16.0 mm
- net GND: track 228.1 -> 235.6 mm, vias 11 -> 12
- net VDD: track 127.9 -> 133.9 mm, vias 3 -> 4
- net N$48: track 2.18 -> 8.12 mm
- net N$45: track 1.63 -> 7.38 mm
- net N$47: track 0.00 -> 2.96 mm
- net N$35: track 6.14 -> 9.00 mm
- net N$15: track 10.7 -> 13.1 mm
- net N$19: track 0.00 -> 2.40 mm
- net N$46: track 2.38 -> 0.00 mm
- net N$8: track 22.7 -> 23.9 mm
- added copper zone on layer 16, net GND

Commit message: TBX01 v0.2-r201508201618
Parts:
- moved C8 0.25 mm to (32.5, 26.3)
Routing:
- net GND: track 235.6 -> 247.9 mm
- net N$23: track 36.2 -> 25.5 mm
- net N$46: track 0.00 -> 7.98 mm
- net N$56: track 0.00 -> 5.08 mm
Changed lines of the file:
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@@
 <element name="C22" library="microbuilder" package="0603" value="100nF" x="44.7548" y="1.9812" rot="R90"/>
 <element name="R17" library="microbuilder" package="0603" value="680" x="46.8376" y="24.257" rot="MR180"/>
-<element name="C8" library="microbuilder" package="0603" value="100nF" x="32.5374" y="26.5684" rot="MR0"/>
+<element name="C8" library="microbuilder" package="0603" value="100nF" x="32.5374" y="26.3144" rot="MR0"/>
 <element name="C9" library="microbuilder" package="0603" value="33nF" x="35.0012" y="23.0124" rot="MR90"/>
 <element name="C23" library="microbuilder" package="0603" value="100nF" x="72.39" y="38.608"/>
@@
 <wire x1="29.7542" y1="22.4308" x2="31.1124" y2="22.4308" width="0.3048" layer="16"/>
 <wire x1="31.1124" y1="22.4308" x2="31.369" y2="22.1742" width="0.3048" layer="16"/>
-<wire x1="33.3874" y1="26.5684" x2="33.4264" y2="26.5684" width="0.254" layer="16"/>
+<wire x1="33.3874" y1="26.3144" x2="33.4264" y2="26.5684" width="0.254" layer="16"/>
 <wire x1="34.1884" y1="24.9936" x2="33.3502" y2="24.1554" width="0.254" layer="1"/>
 <wire x1="34.1884" y1="24.9936" x2="34.671" y2="24.9936" width="0.254" layer="1"/>
@@
 <via x="34.8488" y="25.1714" extent="1-16" drill="0.6"/>
 <wire x1="34.8488" y1="25.1714" x2="34.7844" y2="25.1714" width="0.254" layer="16"/>
-<wire x1="34.7844" y1="25.1714" x2="33.3874" y2="26.5684" width="0.254" layer="16"/>
 <wire x1="20.4216" y1="33.3348" x2="20.428" y2="33.3412" width="0.254" layer="16"/>
 <polygon width="0.254" layer="16">
@@
 <wire x1="19.7612" y1="31.0642" x2="20.066" y2="31.369" width="0.3048" layer="16"/>
 <wire x1="22.5552" y1="33.2734" x2="22.623" y2="33.3412" width="0.3048" layer="16"/>
+<wire x1="1.576" y1="22.334" x2="3.5126" y2="22.334" width="1.27" layer="16"/>
+<wire x1="3.5126" y1="22.334" x2="6.0706" y2="24.892" width="1.27" layer="16"/>
+<wire x1="6.0706" y1="24.892" x2="6.0706" y2="30.607" width="1.27" layer="16"/>
+<wire x1="6.0706" y1="30.607" x2="6.6802" y2="31.2166" width="1.27" layer="16"/>
+<wire x1="33.3874" y1="26.3144" x2="33.7058" y2="26.3144" width="0.3048" layer="16"/>
+<wire x1="33.7058" y1="26.3144" x2="34.8488" y2="25.1714" width="0.3048" layer="16"/>
 <wire x1="71.54" y1="45.72" x2="71.54" y2="70.612" width="0" layer="19" extent="1-1"/>
 <wire x1="71.54" y1="38.608" x2="71.54" y2="45.72" width="0" layer="19" extent="1-1"/>
@@
 <wire x1="16.0782" y1="24.7904" x2="15.2146" y2="23.5712" width="0" layer="19" extent="1-1"/>
 <wire x1="35.0012" y1="22.1624" x2="37.4168" y2="22.4308" width="0" layer="19" extent="16-16"/>
-<wire x1="33.566" y1="28.7958" x2="33.3874" y2="26.5684" width="0" layer="19" extent="16-16"/>
+<wire x1="33.566" y1="28.7958" x2="33.4264" y2="26.5684" width="0" layer="19" extent="16-16"/>
 <wire x1="1.603" y1="24.7914" x2="1.576" y2="22.334" width="0" layer="19" extent="1-16"/>
 <wire x1="44.7548" y1="1.1312" x2="43.2308" y2="3.3528" width="0" layer="19" extent="1-16"/>
@@
 <wire x1="31.9024" y1="17.1958" x2="31.9024" y2="20.2184" width="0.254" layer="16"/>
 <wire x1="47.74" y1="22.1234" x2="47.74" y2="22.1368" width="0.254" layer="16"/>
-<wire x1="47.74" y1="22.1368" x2="48.6664" y2="23.0632" width="0.254" layer="16"/>
-<wire x1="48.6664" y1="23.0632" x2="44.704" y2="23.0632" width="0.254" layer="16"/>
-<wire x1="44.704" y1="23.0632" x2="40.894" y2="26.8732" width="0.254" layer="16"/>
+<wire x1="47.74" y1="22.1368" x2="48.6664" y2="23.0632" width="0" layer="19" extent="1-16"/>
+<wire x1="48.6664" y1="23.0632" x2="44.704" y2="23.0632" width="0" layer="19" extent="1-16"/>
+<wire x1="44.704" y1="23.0632" x2="40.894" y2="26.8732" width="0" layer="19" extent="1-16"/>
 <wire x1="28.2956" y1="14.4018" x2="29.2608" y2="14.4018" width="0.254" layer="16"/>
 <via x="29.2608" y="14.4018" extent="1-16" drill="0.6"/>
@@
 <contactref element="U1" pad="2"/>
 <contactref element="C8" pad="2"/>
-<wire x1="29.7542" y1="25.4308" x2="30.5498" y2="25.4308" width="0.3048" layer="16"/>
-<wire x1="30.5498" y1="25.4308" x2="31.6874" y2="26.5684" width="0.3048" layer="16"/>
+<wire x1="29.7542" y1="25.4308" x2="30.8038" y2="25.4308" width="0.3048" layer="16"/>
+<wire x1="30.8038" y1="25.4308" x2="31.6874" y2="26.3144" width="0.3048" layer="16"/>
 </signal>
 <signal name="N$20">
@@
 <contactref element="U1" pad="21"/>
 <contactref element="B1" pad="4"/>
-<wire x1="20.2612" y1="29.5228" x2="20.2612" y2="28.202" width="0.254" layer="16"/>
-<wire x1="20.2612" y1="28.202" x2="24.0284" y2="24.4348" width="0.254" layer="16"/>
-<wire x1="24.0284" y1="24.4348" x2="24.7502" y2="24.4348" width="0.254" layer="16"/>
 <wire x1="24.7502" y1="24.4348" x2="24.7542" y2="24.4308" width="0.254" layer="16"/>
+<wire x1="20.2692" y1="29.5148" x2="20.2612" y2="29.5228" width="0.254" layer="16"/>
+<wire x1="20.2692" y1="29.5148" x2="20.2692" y2="27.7114" width="0.254" layer="16"/>
+<wire x1="20.2692" y1="27.7114" x2="23.5458" y2="24.4348" width="0.254" layer="16"/>
+<wire x1="23.5458" y1="24.4348" x2="24.7502" y2="24.4348" width="0.254" layer="16"/>
 </signal>
 <signal name="N$46">
 <contactref element="U1" pad="22"/>
 <contactref element="B1" pad="3"/>
-<wire x1="24.7542" y1="24.9308" x2="20.2612" y2="30.5228" width="0" layer="19" extent="16-16"/>
+<wire x1="20.2612" y1="30.5228" x2="20.455" y2="30.5228" width="0.3048" layer="16"/>
+<wire x1="20.455" y1="30.5228" x2="21.0312" y2="29.9466" width="0.3048" layer="16"/>
+<wire x1="21.0312" y1="29.9466" x2="21.0312" y2="27.94" width="0.3048" layer="16"/>
+<wire x1="21.0312" y1="27.94" x2="24.0284" y2="24.9428" width="0.3048" layer="16"/>
+<wire x1="24.0284" y1="24.9428" x2="24.7422" y2="24.9428" width="0.3048" layer="16"/>
+<wire x1="24.7422" y1="24.9428" x2="24.7542" y2="24.9308" width="0.3048" layer="16"/>
 </signal>
 <signal name="N$47">
@@
 <contactref element="B1" pad="5"/>
 <contactref element="C17" pad="2"/>
-<wire x1="19.7612" y1="29.5228" x2="19.7612" y2="28.1432" width="0.254" layer="16"/>
-<wire x1="19.7612" y1="28.1432" x2="23.9776" y2="23.9268" width="0.254" layer="16"/>
-<wire x1="23.9776" y1="23.9268" x2="24.7502" y2="23.9268" width="0.254" layer="16"/>
 <wire x1="24.7502" y1="23.9268" x2="24.7542" y2="23.9308" width="0.254" layer="16"/>
+<wire x1="24.7502" y1="23.9268" x2="23.368" y2="23.9268" width="0.254" layer="16"/>
+<wire x1="23.368" y1="23.9268" x2="19.7612" y2="27.5336" width="0.254" layer="16"/>
+<wire x1="19.7612" y1="27.5336" x2="19.7612" y2="29.5228" width="0.254" layer="16"/>
 <wire x1="19.7612" y1="29.5228" x2="22.5942" y2="29.7942" width="0" layer="19" extent="16-16"/>
 </signal>
@@
 <signal name="N$55">
 </signal>
+<signal name="N$56">
+<wire x1="34.3916" y1="32.3088" x2="34.8234" y2="32.3088" width="0.6096" layer="16"/>
+<wire x1="34.8234" y1="32.3088" x2="34.8234" y2="27.6606" width="0.6096" layer="16"/>
+</signal>
 </signals>

Commit message: TBX01 v0.3
Button update
Parts:
- removed S1, S2: SWITCH-MOMENTARY-2SMD-3, SparkFun-Electromechanical:TACTILE_SWITCH_SMD-3
- removed SW1, SW2, SW3, SW4: SW-TACTILE-PTS840P, we-switch:SW_PTS840P
- added B2, B3, B4, B5, B6, B7: (no value), alps:SKSCLDE010
- moved R19 6.02 mm to (16.3, 36.2)
- moved C20 5.23 mm to (3.94, 7.24), turned to 270 degrees
- moved C22 5.17 mm to (45.6, 7.09)
- moved C21 4.87 mm to (47.8, 34.7)
- moved C18 3.02 mm to (1.07, 22.5)
- moved D1 2.21 mm to (8.71, 30.2)
- moved LED2 1.75 mm to (45.2, 26.0)
- moved LED1 1.66 mm to (45.3, 29.8)
- moved LED3 1.40 mm to (45.6, 22.2)
- moved R8 1.40 mm to (45.4, 28.1)
- moved R17 1.20 mm to (45.6, 24.2)
- moved R15 1.19 mm to (45.7, 20.2)
Connections:
- net GND: now also B2.3, B3.3, B4.3, B5.3, B6.3, B7.3; no longer S1.4, S2.4, SW1.4, SW2.4, SW3.4, SW4.4
- net N$10: now also B7.1; no longer S2.1
- net N$38: now also B3.1; no longer SW1.2
- net N$40: now also B5.1; no longer SW2.2
- net N$41: now also B2.1; no longer SW3.2
- net N$42: now also B4.1; no longer SW4.2
- net N$54: now also B6.1; no longer S1.1
Routing:
- net BAT-PWRGOOD: track 4.79 -> 42.2 mm
- net N$17: track 60.1 -> 24.6 mm
- net BAT-STAT2: track 0.00 -> 30.4 mm, vias 0 -> 1
- net BAT-STAT1: track 10.4 -> 33.1 mm
- net N$54: track 37.9 -> 49.2 mm
- net N$10: track 0.00 -> 9.38 mm
- net N$16: track 24.4 -> 16.7 mm
- net N$43: track 35.6 -> 34.1 mm
- net GND: track 247.9 -> 246.3 mm

Commit message: TBX01 v0.3-r201508201530
Parts:
- removed U$44: INVERTED_F_ANTENNA+0, TI_antenna:DN007+0
- moved C22 5.39 mm to (47.9, 2.21)
Connections:
- net GND: no longer U$44.GND, U$44.GND@1
- net N$47: no longer U$44.FEED
Routing:
- net N$16: track 16.7 -> 45.0 mm
- net N$56: track 5.08 -> 12.1 mm
- net BAT-PWRGOOD: track 42.2 -> 35.3 mm
- net GND: track 246.3 -> 242.6 mm
- net N$47: track 2.96 -> 0.03 mm
- net BAT-STAT1: track 33.1 -> 31.8 mm

Commit message: TBX01 v0.3-r201508230020
Parts:
- added U$44: INVERTED_F_ANTENNA+0, TI_antenna:DN007+0
- moved R19 17.1 mm to (33.2, 34.2), flipped to the bottom
- moved R13 15.6 mm to (46.5, 38.1)
- moved D1 8.47 mm to (16.7, 33.0), turned to 0 degrees
- moved C21 6.88 mm to (46.1, 28.0)
- moved C20 4.35 mm to (1.75, 11.0), turned to 0 degrees
- moved R12 3.02 mm to (39.6, 34.0)
- moved C17 2.82 mm to (21.4, 31.7), flipped to the top, turned to 180 degrees
- moved B1 1.37 mm to (20.0, 31.4), turned to 90 degrees
- moved JP2 0.99 mm to (9.17, 3.53)
- moved R11 0.88 mm to (39.2, 3.10)
- moved C27 0.23 mm to (29.4, 28.9)
Connections:
- net GND: now also U$44.GND, U$44.GND@1
- net N$47: now also U$44.FEED
Routing:
- net N$10: track 9.38 -> 71.8 mm, vias 0 -> 3
- net N$54: track 49.2 -> 92.8 mm
- net N$17: track 24.6 -> 52.7 mm, vias 2 -> 3
- net N$16: track 45.0 -> 28.4 mm
- net N$15: track 13.1 -> 0.00 mm
- net DCDC-PWRGOOD: track 32.7 -> 23.8 mm
- net VDD: track 133.9 -> 142.6 mm, vias 4 -> 6
- net N$56: track 12.1 -> 5.18 mm
- net N$40: track 0.00 -> 6.49 mm
- net N$48: track 8.48 -> 14.8 mm, vias 0 -> 1
- net GND: track 242.6 -> 236.8 mm, vias 12 -> 13
- net N$25: track 29.6 -> 33.8 mm
- net BAT-PWRGOOD: track 35.3 -> 31.4 mm, vias 1 -> 0
- net VBAT: track 40.2 -> 36.6 mm
- net N$14: track 2.97 -> 0.00 mm
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- removed copper zone on layer 16, net GND

Commit message: TBX01 v0.3-r201508230138
Parts:
- moved B1 1.27 mm to (18.7, 31.3)
Routing:
- net GND: track 236.8 -> 256.0 mm
- net VDD: track 142.6 -> 153.9 mm
- net N$48: track 14.8 -> 16.3 mm
- net N$46: track 8.42 -> 9.58 mm
- net N$45: track 10.2 -> 10.8 mm

Commit message: TBX01 v0.3-r201508231801
Parts:
- moved R2 87.1 mm to (9.98, 9.22)
- moved R3 87.0 mm to (9.93, 7.54)
- moved R4 86.9 mm to (9.98, 5.89)
- moved C5 54.9 mm to (45.9, 22.5), turned to 90 degrees
- moved C23 48.8 mm to (24.5, 29.7), flipped to the bottom, turned to 270 degrees
- moved C25 46.4 mm to (26.9, 25.9), turned to 180 degrees
- moved C24 44.0 mm to (30.3, 24.2), turned to 90 degrees
- moved C19 41.1 mm to (45.7, 14.5), flipped to the bottom, turned to 90 degrees
- moved R18 37.0 mm to (21.9, 29.3)
- moved C22 26.0 mm to (45.9, 28.2)
- moved R19 24.0 mm to (11.0, 25.0), turned to 90 degrees
- moved C21 20.9 mm to (45.8, 7.14)
- moved R12 5.34 mm to (44.9, 34.1), turned to 0 degrees
- moved C17 2.88 mm to (18.8, 30.3), turned to 270 degrees
- moved R13 2.25 mm to (45.1, 36.4), turned to 0 degrees
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Routing:
- net GND: track 256.0 -> 305.3 mm, vias 13 -> 16
- net VDD: track 153.9 -> 192.8 mm, vias 6 -> 9
- net N$23: track 25.5 -> 52.7 mm, vias 3 -> 6
- net N$17: track 52.7 -> 62.7 mm, vias 3 -> 4
- net N$54: track 92.8 -> 83.2 mm
- net N$38: track 0.00 -> 8.63 mm
- net N$15: track 0.00 -> 7.49 mm
- net N$14: track 0.00 -> 5.53 mm
- net N$49: track 0.00 -> 4.57 mm
- net N$48: track 16.3 -> 12.3 mm, vias 1 -> 0
- net BAT-STAT2: track 29.9 -> 27.1 mm
- net BAT-STAT1: track 31.7 -> 29.0 mm
- net BAT-PWRGOOD: track 31.4 -> 28.7 mm
- net N$16: track 28.4 -> 25.7 mm
- net N$36: track 16.0 -> 18.3 mm
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