File: TBX01.brd (EAGLE design)
At the start: 49.8 x 40.1 mm, 75 parts, among them IC1 TPS62120, U3 STM32L151CCT6, U6 MCP73833, X2 FH12-10S-0.5SH, Y1 CRYSTAL.ABS07

Commit message: TBX01 v0.3-r201508240212
Parts:
- moved R7 73.1 mm to (14.1, 15.2), flipped to the bottom, turned to 270 degrees
- moved C5 11.8 mm to (47.9, 10.9), turned to 180 degrees
- moved C19 5.72 mm to (45.7, 20.2), flipped to the top, turned to 270 degrees
- moved R3 4.70 mm to (11.2, 12.1)
- moved C21 4.22 mm to (47.9, 3.45), turned to 0 degrees
- moved R4 3.07 mm to (11.3, 8.69)
- moved R2 1.71 mm to (11.2, 10.4)
- moved C18 1.21 mm to (1.68, 23.6)
- moved C20 1.10 mm to (1.14, 11.9), turned to 90 degrees
- moved R10 1.07 mm to (42.5, 7.59)
- moved C26 0.48 mm to (29.4, 30.7)
- moved C9 0.46 mm to (34.5, 23.0)
- moved C22 0.40 mm to (45.7, 27.8), turned to 270 degrees
- moved C8 0.38 mm to (33.0, 26.4)
- moved C27 0.23 mm to (29.4, 29.1)
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Connections:
- net GND: now also B2.1, B2.2, B3.1, B3.2, B4.1, B4.2, B5.1, B5.2, B6.1, B6.2, B7.1, B7.2; no longer B2.3, B3.3, B4.3, B5.3, B6.3, B7.3
- net N$10: now also B7.3, B7.4; no longer B7.1
- net N$38: now also B3.3, B3.4; no longer B3.1
- net N$40: now also B5.3, B5.4; no longer B5.1
- net N$41: now also B2.3, B2.4; no longer B2.1
- net N$42: now also B4.3, B4.4; no longer B4.1
- net N$54: now also B6.3, B6.4; no longer B6.1
Routing:
- net GND: track 305.3 -> 352.2 mm, vias 16 -> 19
- net N$40: track 6.49 -> 33.1 mm, vias 0 -> 2
- net N$54: track 83.2 -> 57.6 mm
- net BAT-PWRGOOD: track 28.7 -> 49.2 mm, vias 0 -> 1
- net N$10: track 70.6 -> 50.1 mm
- net VBAT: track 36.6 -> 53.2 mm
- net BAT-STAT1: track 29.0 -> 42.7 mm
- net N$41: track 0.00 -> 13.2 mm, vias 0 -> 1
- net BAT-STAT2: track 27.1 -> 40.1 mm
- net N$56: track 5.18 -> 0.00 mm
- net DCDC-PWRGOOD: track 23.8 -> 27.9 mm
- net N$37: track 0.00 -> 2.31 mm
- net N$44: track 0.00 -> 1.93 mm
- net N$24: track 15.6 -> 17.4 mm
- net VDD: track 192.8 -> 191.0 mm
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- added copper zone on layer 16, net GND

Commit message: TBX01 v0.3-r201508241143
Parts:
- moved C22 3.98 mm to (47.9, 24.5), turned to 180 degrees
- moved C18 0.91 mm to (1.88, 24.5), turned to 0 degrees
- moved C21 0.20 mm to (47.9, 3.66), turned to 180 degrees
Routing:
- net GND: track 352.2 -> 392.5 mm
- net N$54: track 57.6 -> 96.2 mm
- net N$10: track 50.1 -> 72.8 mm
- net N$41: track 13.2 -> 25.5 mm, vias 1 -> 2
- net N$40: track 33.1 -> 22.5 mm
- net N$38: track 10.3 -> 17.3 mm
- net N$42: track 0.00 -> 4.95 mm
- net N$16: track 25.7 -> 29.2 mm
- net VDD: track 191.0 -> 193.2 mm
- net VIN: track 15.2 -> 15.8 mm

Commit message: TBX01 v0.4
Parts:
- removed U$1: LS013B4DN04, sharp_LCD:DISPLAY1
- moved D1 6.82 mm to (23.5, 32.1)
- moved C20 0.43 mm to (1.57, 11.9)
- moved R4 0.10 mm to (11.2, 8.69)
- moved C10 0.08 mm to (23.8, 24.3)
Routing:
- net N$16: track 29.2 -> 126.1 mm, vias 0 -> 4
- net N$42: track 4.95 -> 76.5 mm, vias 0 -> 4
- net N$38: track 17.3 -> 65.7 mm, vias 1 -> 4
- net GND: track 392.5 -> 427.3 mm, vias 19 -> 18
- net VDD: track 193.2 -> 206.8 mm, vias 9 -> 10
- net N$41: track 25.5 -> 35.1 mm
- net N$17: track 62.7 -> 53.2 mm, vias 4 -> 2
- net N$54: track 96.2 -> 89.1 mm
- net N$40: track 22.5 -> 29.4 mm
- net N$10: track 72.8 -> 67.1 mm
- net VBAT: track 53.2 -> 50.2 mm
- net N$2: track 0.00 -> 1.65 mm
- net N$48: track 12.3 -> 13.8 mm, vias 0 -> 1

Commit message: TBX01 v0.4-r201508241723
Parts:
- moved C12 0.89 mm to (24.2, 16.5)
- moved L1 0.53 mm to (23.6, 2.82)
- moved C17 0.13 mm to (18.8, 30.4)
- moved R8 0.08 mm to (45.3, 28.2)
Connections:
- net TP: now also U1.GND; no longer U1.33
Routing:
- net GND: track 427.3 -> 428.8 mm

Commit message: TBX01 v0.5
Parts:
- moved C22 0.18 mm to (47.9, 24.7)
Routing:
- net N$38: track 65.5 -> 65.0 mm
- net VDD: track 206.5 -> 206.0 mm

Commit message: TBX01 v0.6
Parts:
- JP1: value USB-MICROB -> USB-RECEPTABLE-HIROSE-ZX62-AB-5PA(11); device SparkFun-Connectors:USB-MICROB -> daspilker:HIROSE-ZX62-AB-5PA(11)
- moved JP1 1.54 mm to (0.30, 19.2), flipped to the top, turned to 270 degrees
Connections:
- removed net TP: U1.GND
- net D+: now also JP1.P$4; no longer JP1.D+
- net D-: now also JP1.P$2; no longer JP1.D-
- net GND: now also JP1.P$5, U1.GND; no longer JP1.GND, JP1.MT1, JP1.MT2
- net VIN: now also JP1.P$1; no longer JP1.VBUS
Routing:
- net GND: track 429.0 -> 432.4 mm, vias 18 -> 19
- net N$40: track 29.8 -> 31.8 mm
- net D+: track 21.5 -> 19.6 mm
- net BAT-STAT1: track 42.7 -> 44.2 mm
- net BAT-PWRGOOD: track 49.1 -> 50.5 mm
- net N$36: track 18.3 -> 17.3 mm
- net VIN: track 15.8 -> 16.8 mm
- net N$16: track 126.1 -> 125.3 mm
- net D-: track 22.8 -> 22.1 mm
- added copper zone on layer 16, net N$56
- added copper zone on layer 16, net N$57

Commit message: TBX01 v0.7
Routing:
- net GND: track 432.4 -> 436.7 mm
Changed lines of the file:
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@@
 <via x="34.8488" y="25.1714" extent="1-16" drill="0.6"/>
 <wire x1="34.8488" y1="25.1714" x2="34.7844" y2="25.1714" width="0.254" layer="16"/>
-<wire x1="6.0706" y1="24.892" x2="6.0706" y2="30.607" width="1.27" layer="16"/>
+<wire x1="6.0706" y1="21.7678" x2="6.0706" y2="30.607" width="1.27" layer="16"/>
 <wire x1="6.0706" y1="30.607" x2="6.6802" y2="31.2166" width="1.27" layer="16"/>
 <contactref element="B3" pad="1"/>
@@
 <wire x1="10.8966" y1="20.0152" x2="9.1186" y2="18.2372" width="0.4064" layer="1"/>
 <via x="9.1186" y="18.2372" extent="1-16" drill="0.6"/>
+<wire x1="6.0706" y1="21.7678" x2="6.0706" y2="20.6248" width="0.6096" layer="16"/>
 </signal>
 <signal name="VDD">

Commit message: TBX01 v1.0
Parts:
- C1: value 1 uF -> 1uF
- C2, C3: value 4.7 uF -> 4.7uF
- C4: value 15 pF -> 15pF
- R1: value 14 kOhms -> 14k
- R2: value 4.7 kOhms -> 4.7k
- R3, R4, R7: value 4.7kOhms -> 4.7k
- R5: value 510 kOhms -> 510k
- R6: value 180 kOhms -> 180k
Other:
- board text added: "TBX01 v1.0 27/08/2015 Tomasz Bialas"
Changed lines of the file:
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@@
 <hole x="2.3114" y="36.576" drill="2.8"/>
 <hole x="32.639" y="6.0706" drill="2.8"/>
+<text x="4.4196" y="33.7312" size="0.6096" layer="25" font="vector">TBX01 v1.0
+27/08/2015 Tomasz Bialas</text>
 </plain>
 <attributes>
@@
 <attribute name="NAME" x="5.08" y="10.9728" size="0.8128" layer="26" ratio="18" rot="MR180"/>
 </element>
-<element name="C1" library="rcl" package="C0603" value="1 uF" x="4.826" y="5.842" smashed="yes" rot="MR270">
+<element name="C1" library="rcl" package="C0603" value="1uF" x="4.826" y="5.842" smashed="yes" rot="MR270">
 <attribute name="NAME" x="5.3086" y="10.2616" size="1.27" layer="26" rot="MR270"/>
 </element>
-<element name="C2" library="rcl" package="C0603" value="4.7 uF" x="13.97" y="4.826" smashed="yes" rot="MR0">
+<element name="C2" library="rcl" package="C0603" value="4.7uF" x="13.97" y="4.826" smashed="yes" rot="MR0">
 <attribute name="NAME" x="15.0114" y="5.842" size="1.27" layer="26" rot="MR0"/>
 </element>
-<element name="R1" library="microbuilder" package="0603" value="14 kOhms" x="10.668" y="8.128" smashed="yes" rot="MR90">
+<element name="R1" library="microbuilder" package="0603" value="14k" x="10.668" y="8.128" smashed="yes" rot="MR90">
 <attribute name="NAME" x="10.3124" y="10.16" size="0.8128" layer="26" font="vector" ratio="18" rot="MR90"/>
 </element>
-<element name="R2" library="microbuilder" package="0603" value="4.7 kOhms" x="11.2268" y="10.3886" smashed="yes">
+<element name="R2" library="microbuilder" package="0603" value="4.7k" x="11.2268" y="10.3886" smashed="yes">
 <attribute name="NAME" x="13.208" y="10.3124" size="0.8128" layer="25" font="vector" ratio="18"/>
 </element>
-<element name="R3" library="microbuilder" package="0603" value="4.7kOhms" x="11.2014" y="12.065" smashed="yes">
+<element name="R3" library="microbuilder" package="0603" value="4.7k" x="11.2014" y="12.065" smashed="yes">
 <attribute name="NAME" x="12.9794" y="11.938" size="0.8128" layer="25" font="vector" ratio="18"/>
 </element>
-<element name="R4" library="microbuilder" package="0603" value="4.7kOhms" x="11.1506" y="8.6868" smashed="yes">
+<element name="R4" library="microbuilder" package="0603" value="4.7k" x="11.1506" y="8.6868" smashed="yes">
 <attribute name="NAME" x="7.8994" y="8.3312" size="0.8128" layer="25" font="vector" ratio="18"/>
 </element>
@@
 <attribute name="NAME" x="26.34" y="7.5154" size="0.8128" layer="26" rot="MR270"/>
 </element>
-<element name="C3" library="rcl" package="C0603" value="4.7 uF" x="29.464" y="10.414" smashed="yes" rot="MR0">
+<element name="C3" library="rcl" package="C0603" value="4.7uF" x="29.464" y="10.414" smashed="yes" rot="MR0">
 <attribute name="NAME" x="32.385" y="9.8806" size="0.6096" layer="26" rot="MR0"/>
 </element>
@@
 <attribute name="NAME" x="22.822" y="2.3194" size="0.4064" layer="26" rot="MR180"/>
 </element>
-<element name="C4" library="rcl" package="C0603" value="15 pF" x="28.448" y="4.826" smashed="yes" rot="MR0">
+<element name="C4" library="rcl" package="C0603" value="15pF" x="28.448" y="4.826" smashed="yes" rot="MR0">
 <attribute name="NAME" x="29.718" y="5.9436" size="0.6096" layer="26" rot="MR0"/>
 </element>
-<element name="R5" library="microbuilder" package="0603" value="510 kOhms" x="28.448" y="2.794" smashed="yes" rot="MR180">
+<element name="R5" library="microbuilder" package="0603" value="510k" x="28.448" y="2.794" smashed="yes" rot="MR180">
 <attribute name="NAME" x="30.226" y="2.921" size="0.8128" layer="26" font="vector" ratio="18" rot="MR180"/>
 </element>
-<element name="R6" library="microbuilder" package="0603" value="180 kOhms" x="27.5844" y="8.4582" smashed="yes" rot="MR180">
+<element name="R6" library="microbuilder" package="0603" value="180k" x="27.5844" y="8.4582" smashed="yes" rot="MR180">
 <attribute name="NAME" x="29.3624" y="8.5852" size="0.8128" layer="26" font="vector" ratio="18" rot="MR180"/>
 </element>
-<element name="R7" library="microbuilder" package="0603" value="4.7kOhms" x="14.1224" y="15.1892" smashed="yes" rot="MR270">
+<element name="R7" library="microbuilder" package="0603" value="4.7k" x="14.1224" y="15.1892" smashed="yes" rot="MR270">
 <attribute name="NAME" x="14.2494" y="13.4112" size="0.8128" layer="26" font="vector" ratio="18" rot="MR270"/>
 </element>
@@
 </board>
 </drawing>
+<compatibility>
+<note version="6.3" minversion="6.2.2" severity="warning">
+Since Version 6.2.2 text objects can contain more than one line,
+which will not be processed correctly with this version.
+</note>
+</compatibility>
 </eagle>
