File: TBX01.sch (EAGLE design)
At the start: 75 parts, among them IC1 TPS62120, SW1 SW-TACTILE-PTS840P, SW2 SW-TACTILE-PTS840P, SW3 SW-TACTILE-PTS840P, SW4 SW-TACTILE-PTS840P, U3 STM32L151CCT6, U6 MCP73833, X2 FH12-10S-0.5SH, Y1 CRYSTAL.ABS07

Commit message: TBX01 v0.2
Parts:
- removed C13: 10uF, microbuilder:CAP_CERAMIC0603
- added D1: (no value), microbuilder:DIODESMA
Connections:
- new net N$54: C5.P$2, D1.A, JTAG1.15, S1.1, U3.NRST
- net GND: no longer C13.P$2
- net N$10: now also D1.C; no longer C5.P$2, JTAG1.15, S1.1, U3.NRST
- net VDD: no longer C13.P$1
Changed lines of the file:
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@@
 <part name="U$27" library="microbuilder" deviceset="VDD" device=""/>
 <part name="U$29" library="microbuilder" deviceset="GND" device=""/>
-<part name="U$30" library="microbuilder" deviceset="VDD" device=""/>
-<part name="U$31" library="microbuilder" deviceset="GND" device=""/>
-<part name="C13" library="microbuilder" deviceset="CAP_CERAMIC" device="0603" value="10uF"/>
 <part name="U$32" library="microbuilder" deviceset="VBAT" device=""/>
 <part name="U$33" library="microbuilder" deviceset="GND" device=""/>
@@
 <part name="R22" library="microbuilder" deviceset="RESISTOR" device="0603" value="4.7k"/>
 <part name="R23" library="microbuilder" deviceset="RESISTOR" device="0603" value="4.7k"/>
+<part name="D1" library="microbuilder" deviceset="DIODE" device="SMA"/>
 </parts>
 <sheets>
@@
 <instance part="U$27" gate="G$1" x="-106.68" y="109.22"/>
 <instance part="U$29" gate="G$1" x="-106.68" y="86.36"/>
-<instance part="U$30" gate="G$1" x="83.82" y="172.72"/>
-<instance part="U$31" gate="G$1" x="83.82" y="149.86"/>
-<instance part="C13" gate="G$1" x="83.82" y="160.02"/>
 <instance part="U$32" gate="G$1" x="-38.1" y="177.8"/>
 <instance part="U$33" gate="G$1" x="-48.26" y="-66.04"/>
@@
 <instance part="R22" gate="G$1" x="48.26" y="93.98" rot="R90"/>
 <instance part="R23" gate="G$1" x="53.34" y="88.9" rot="R90"/>
+<instance part="D1" gate="G$1" x="25.4" y="96.52" rot="R90"/>
 </instances>
 <busses>
@@
 <pinref part="U$29" gate="G$1" pin="GND"/>
 <wire x1="-106.68" y1="91.44" x2="-106.68" y2="88.9" width="0.1524" layer="91"/>
-</segment>
-<segment>
-<pinref part="C13" gate="G$1" pin="P$2"/>
-<pinref part="U$31" gate="G$1" pin="GND"/>
-<wire x1="83.82" y1="157.48" x2="83.82" y2="152.4" width="0.1524" layer="91"/>
 </segment>
 <segment>
@@
 </segment>
 <segment>
-<pinref part="U$30" gate="G$1" pin="VDD"/>
-<pinref part="C13" gate="G$1" pin="P$1"/>
-<wire x1="83.82" y1="170.18" x2="83.82" y2="165.1" width="0.1524" layer="91"/>
-</segment>
-<segment>
 <pinref part="X2" gate="-7" pin="1"/>
 <pinref part="U$6" gate="G$1" pin="VDD"/>
@@
 <junction x="134.62" y="76.2"/>
 <wire x1="154.94" y1="76.2" x2="154.94" y2="139.7" width="0.1524" layer="91"/>
-<pinref part="U3" gate="A" pin="NRST"/>
-<wire x1="-2.54" y1="55.88" x2="17.78" y2="55.88" width="0.1524" layer="91"/>
-<wire x1="17.78" y1="55.88" x2="17.78" y2="127" width="0.1524" layer="91"/>
-<wire x1="17.78" y1="127" x2="-149.86" y2="127" width="0.1524" layer="91"/>
-<wire x1="-149.86" y1="127" x2="-149.86" y2="76.2" width="0.1524" layer="91"/>
-<pinref part="JTAG1" gate="G$1" pin="15"/>
-<wire x1="-149.86" y1="76.2" x2="-172.72" y2="76.2" width="0.1524" layer="91"/>
-<wire x1="17.78" y1="55.88" x2="25.4" y2="55.88" width="0.1524" layer="91"/>
-<junction x="17.78" y="55.88"/>
-<pinref part="C5" gate="G$1" pin="P$2"/>
-<pinref part="S1" gate="G$1" pin="1"/>
-<wire x1="25.4" y1="55.88" x2="27.94" y2="55.88" width="0.1524" layer="91"/>
-<junction x="27.94" y="55.88"/>
-<wire x1="25.4" y1="55.88" x2="25.4" y2="134.62" width="0.1524" layer="91"/>
-<junction x="25.4" y="55.88"/>
+<wire x1="25.4" y1="99.06" x2="25.4" y2="134.62" width="0.1524" layer="91"/>
 <wire x1="25.4" y1="134.62" x2="119.38" y2="134.62" width="0.1524" layer="91"/>
 <pinref part="S2" gate="G$1" pin="1"/>
@@
 <wire x1="119.38" y1="139.7" x2="119.38" y2="134.62" width="0.1524" layer="91"/>
 <junction x="119.38" y="134.62"/>
+<pinref part="D1" gate="G$1" pin="C"/>
 </segment>
 </net>
@@
 </segment>
 </net>
+<net name="N$54" class="0">
+<segment>
+<pinref part="JTAG1" gate="G$1" pin="15"/>
+<wire x1="-149.86" y1="76.2" x2="-172.72" y2="76.2" width="0.1524" layer="91"/>
+<pinref part="D1" gate="G$1" pin="A"/>
+<pinref part="C5" gate="G$1" pin="P$2"/>
+<pinref part="S1" gate="G$1" pin="1"/>
+<junction x="27.94" y="55.88"/>
+<wire x1="25.4" y1="55.88" x2="27.94" y2="55.88" width="0.1524" layer="91"/>
+<wire x1="25.4" y1="55.88" x2="25.4" y2="93.98" width="0.1524" layer="91"/>
+<junction x="25.4" y="55.88"/>
+<pinref part="U3" gate="A" pin="NRST"/>
+<wire x1="-2.54" y1="55.88" x2="17.78" y2="55.88" width="0.1524" layer="91"/>
+<wire x1="17.78" y1="55.88" x2="25.4" y2="55.88" width="0.1524" layer="91"/>
+<junction x="17.78" y="55.88"/>
+<wire x1="17.78" y1="55.88" x2="17.78" y2="127" width="0.1524" layer="91"/>
+<wire x1="17.78" y1="127" x2="-149.86" y2="127" width="0.1524" layer="91"/>
+<wire x1="-149.86" y1="127" x2="-149.86" y2="76.2" width="0.1524" layer="91"/>
+</segment>
+</net>

Commit message: TBX01 v0.2-r201508171545
On branch master
	.~lock.TBX-01_power.ods#
nothing added to commit but untracked files present (use "git add" to track)
Parts:
- D1: device microbuilder:DIODESMA -> microbuilder:DIODESOD-123
Connections:
- net N$18: now also Y1.2; no longer Y1.1
- net N$22: now also Y1.1; no longer Y1.2
Changed lines of the file:
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@@
 <part name="R22" library="microbuilder" deviceset="RESISTOR" device="0603" value="4.7k"/>
 <part name="R23" library="microbuilder" deviceset="RESISTOR" device="0603" value="4.7k"/>
-<part name="D1" library="microbuilder" deviceset="DIODE" device="SMA"/>
+<part name="D1" library="microbuilder" deviceset="DIODE" device="SOD-123"/>
 </parts>
 <sheets>
@@
 <wire x1="-38.1" y1="10.16" x2="-38.1" y2="2.54" width="0.1524" layer="91"/>
 <pinref part="C6" gate="G$1" pin="P$1"/>
-<pinref part="Y1" gate="G$1" pin="1"/>
+<pinref part="Y1" gate="G$1" pin="2"/>
 <wire x1="-38.1" y1="2.54" x2="-38.1" y2="0" width="0.1524" layer="91"/>
-<wire x1="-38.1" y1="2.54" x2="-35.56" y2="2.54" width="0.1524" layer="91"/>
+<wire x1="-38.1" y1="2.54" x2="-30.48" y2="2.54" width="0.1524" layer="91"/>
 <junction x="-38.1" y="2.54"/>
 </segment>
@@
 <pinref part="C7" gate="G$1" pin="P$1"/>
 <wire x1="-27.94" y1="2.54" x2="-27.94" y2="0" width="0.1524" layer="91"/>
-<pinref part="Y1" gate="G$1" pin="2"/>
-<wire x1="-30.48" y1="2.54" x2="-27.94" y2="2.54" width="0.1524" layer="91"/>
+<pinref part="Y1" gate="G$1" pin="1"/>
+<wire x1="-35.56" y1="2.54" x2="-27.94" y2="2.54" width="0.1524" layer="91"/>
 <junction x="-27.94" y="2.54"/>
 <wire x1="5.08" y1="25.4" x2="5.08" y2="10.16" width="0.1524" layer="91"/>

Commit message: TBX01 v0.2-r201508172343
Connections:
- net GND: now also C11.P$1, C12.P$1; no longer C11.P$2, C12.P$2
- net VDD: now also C11.P$2, C12.P$2; no longer C11.P$1, C12.P$1
Changed lines of the file:
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@@
 <pinref part="C10" gate="G$1" pin="P$2"/>
 <wire x1="-116.84" y1="93.98" x2="-116.84" y2="91.44" width="0.1524" layer="91"/>
-<pinref part="C11" gate="G$1" pin="P$2"/>
+<pinref part="C11" gate="G$1" pin="P$1"/>
 <wire x1="-116.84" y1="91.44" x2="-106.68" y2="91.44" width="0.1524" layer="91"/>
-<wire x1="-106.68" y1="91.44" x2="-106.68" y2="93.98" width="0.1524" layer="91"/>
-<pinref part="C12" gate="G$1" pin="P$2"/>
+<wire x1="-106.68" y1="91.44" x2="-106.68" y2="101.6" width="0.1524" layer="91"/>
+<pinref part="C12" gate="G$1" pin="P$1"/>
 <wire x1="-106.68" y1="91.44" x2="-96.52" y2="91.44" width="0.1524" layer="91"/>
-<wire x1="-96.52" y1="91.44" x2="-96.52" y2="93.98" width="0.1524" layer="91"/>
+<wire x1="-96.52" y1="91.44" x2="-96.52" y2="101.6" width="0.1524" layer="91"/>
 <junction x="-106.68" y="91.44"/>
 <pinref part="U$29" gate="G$1" pin="GND"/>
@@
 </segment>
 <segment>
-<pinref part="C11" gate="G$1" pin="P$1"/>
+<pinref part="C11" gate="G$1" pin="P$2"/>
 <pinref part="U$27" gate="G$1" pin="VDD"/>
-<wire x1="-106.68" y1="101.6" x2="-106.68" y2="104.14" width="0.1524" layer="91"/>
-<pinref part="C12" gate="G$1" pin="P$1"/>
+<wire x1="-106.68" y1="93.98" x2="-106.68" y2="104.14" width="0.1524" layer="91"/>
+<pinref part="C12" gate="G$1" pin="P$2"/>
 <wire x1="-106.68" y1="104.14" x2="-106.68" y2="106.68" width="0.1524" layer="91"/>
-<wire x1="-96.52" y1="101.6" x2="-96.52" y2="104.14" width="0.1524" layer="91"/>
+<wire x1="-96.52" y1="93.98" x2="-96.52" y2="104.14" width="0.1524" layer="91"/>
 <wire x1="-96.52" y1="104.14" x2="-106.68" y2="104.14" width="0.1524" layer="91"/>
 <junction x="-106.68" y="104.14"/>

Commit message: TBX01 v0.2-r201508181630
Connections:
- net GND: now also C12.P$2; no longer C12.P$1
- net VDD: now also C12.P$1; no longer C12.P$2
Changed lines of the file:
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@@
 <wire x1="-116.84" y1="91.44" x2="-106.68" y2="91.44" width="0.1524" layer="91"/>
 <wire x1="-106.68" y1="91.44" x2="-106.68" y2="101.6" width="0.1524" layer="91"/>
-<pinref part="C12" gate="G$1" pin="P$1"/>
+<pinref part="C12" gate="G$1" pin="P$2"/>
 <wire x1="-106.68" y1="91.44" x2="-96.52" y2="91.44" width="0.1524" layer="91"/>
-<wire x1="-96.52" y1="91.44" x2="-96.52" y2="101.6" width="0.1524" layer="91"/>
+<wire x1="-96.52" y1="91.44" x2="-96.52" y2="93.98" width="0.1524" layer="91"/>
 <junction x="-106.68" y="91.44"/>
 <pinref part="U$29" gate="G$1" pin="GND"/>
@@
 <pinref part="U$27" gate="G$1" pin="VDD"/>
 <wire x1="-106.68" y1="93.98" x2="-106.68" y2="104.14" width="0.1524" layer="91"/>
-<pinref part="C12" gate="G$1" pin="P$2"/>
+<pinref part="C12" gate="G$1" pin="P$1"/>
 <wire x1="-106.68" y1="104.14" x2="-106.68" y2="106.68" width="0.1524" layer="91"/>
-<wire x1="-96.52" y1="93.98" x2="-96.52" y2="104.14" width="0.1524" layer="91"/>
+<wire x1="-96.52" y1="101.6" x2="-96.52" y2="104.14" width="0.1524" layer="91"/>
 <wire x1="-96.52" y1="104.14" x2="-106.68" y2="104.14" width="0.1524" layer="91"/>
 <junction x="-106.68" y="104.14"/>

Commit message: TBX01 v0.3
Button update
Parts:
- removed S1, S2: SWITCH-MOMENTARY-2SMD-3, SparkFun-Electromechanical:SWITCH-MOMENTARY-2SMD-3
- removed SW1, SW2, SW3, SW4: SW-TACTILE-PTS840P, we-switch:SW-TACTILE-PTS840P
- added B2, B3, B4, B5, B6, B7: (no value), alps:SKSCLDE010
Connections:
- net GND: now also B2.4, B3.4, B4.4, B5.4, B6.4, B7.4; no longer S1.2, S2.2, SW1.S2, SW2.S2, SW3.S2, SW4.S2
- net N$10: now also B7.1; no longer S2.1
- net N$38: now also B3.1; no longer SW1.P2
- net N$40: now also B5.1; no longer SW2.P2
- net N$41: now also B2.1; no longer SW3.P2
- net N$42: now also B4.1; no longer SW4.P2
- net N$54: now also B6.1; no longer S1.1
Other:
- moved on the sheet: C5

Commit message: TBX01 v0.3-r201508201530
Parts:
- removed U$44: INVERTED_F_ANTENNA+0, TI_antenna:INVERTED_F_ANTENNA+0
Connections:
- net GND: no longer U$44.GND, U$44.GND@1
- net N$47: no longer U$44.FEED
Changed lines of the file:
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@@
 <part name="U$40" library="microbuilder" deviceset="GND" device=""/>
 <part name="U$41" library="microbuilder" deviceset="GND" device=""/>
-<part name="U$44" library="TI_antenna" deviceset="INVERTED_F_ANTENNA" device="+0"/>
 <part name="U$45" library="microbuilder" deviceset="GND" device=""/>
 <part name="C17" library="microbuilder" deviceset="CAP_CERAMIC" device="0603" value="2.2nF"/>
@@
 <instance part="U$40" gate="G$1" x="137.16" y="55.88"/>
 <instance part="U$41" gate="G$1" x="99.06" y="109.22"/>
-<instance part="U$44" gate="G$1" x="152.4" y="20.32" rot="R180"/>
 <instance part="U$45" gate="G$1" x="177.8" y="5.08"/>
 <instance part="C17" gate="G$1" x="142.24" y="50.8" rot="R180"/>
@@
 </segment>
 <segment>
-<pinref part="U$44" gate="G$1" pin="GND"/>
 <wire x1="160.02" y1="22.86" x2="165.1" y2="22.86" width="0.1524" layer="91"/>
 <wire x1="165.1" y1="22.86" x2="177.8" y2="22.86" width="0.1524" layer="91"/>
@@
 <pinref part="B1" gate="G$1" pin="GND"/>
 <wire x1="177.8" y1="58.42" x2="172.72" y2="58.42" width="0.1524" layer="91"/>
-<pinref part="U$44" gate="G$1" pin="GND@1"/>
 <wire x1="160.02" y1="25.4" x2="165.1" y2="25.4" width="0.1524" layer="91"/>
 <wire x1="165.1" y1="25.4" x2="165.1" y2="22.86" width="0.1524" layer="91"/>
@@
 <wire x1="172.72" y1="53.34" x2="175.26" y2="53.34" width="0.1524" layer="91"/>
 <wire x1="175.26" y1="53.34" x2="175.26" y2="17.78" width="0.1524" layer="91"/>
-<pinref part="U$44" gate="G$1" pin="FEED"/>
 <wire x1="175.26" y1="17.78" x2="160.02" y2="17.78" width="0.1524" layer="91"/>
 </segment>

Commit message: TBX01 v0.3-r201508230020
Parts:
- added U$44: INVERTED_F_ANTENNA+0, TI_antenna:INVERTED_F_ANTENNA+0
Connections:
- net GND: now also U$44.GND, U$44.GND@1
- net N$47: now also U$44.FEED
Changed lines of the file:
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@@
 <part name="U$40" library="microbuilder" deviceset="GND" device=""/>
 <part name="U$41" library="microbuilder" deviceset="GND" device=""/>
+<part name="U$44" library="TI_antenna" deviceset="INVERTED_F_ANTENNA" device="+0"/>
 <part name="U$45" library="microbuilder" deviceset="GND" device=""/>
 <part name="C17" library="microbuilder" deviceset="CAP_CERAMIC" device="0603" value="2.2nF"/>
@@
 <instance part="U$40" gate="G$1" x="137.16" y="55.88"/>
 <instance part="U$41" gate="G$1" x="99.06" y="109.22"/>
+<instance part="U$44" gate="G$1" x="152.4" y="20.32" rot="R180"/>
 <instance part="U$45" gate="G$1" x="177.8" y="5.08"/>
 <instance part="C17" gate="G$1" x="142.24" y="50.8" rot="R180"/>
@@
 </segment>
 <segment>
+<pinref part="U$44" gate="G$1" pin="GND"/>
 <wire x1="160.02" y1="22.86" x2="165.1" y2="22.86" width="0.1524" layer="91"/>
 <wire x1="165.1" y1="22.86" x2="177.8" y2="22.86" width="0.1524" layer="91"/>
@@
 <pinref part="B1" gate="G$1" pin="GND"/>
 <wire x1="177.8" y1="58.42" x2="172.72" y2="58.42" width="0.1524" layer="91"/>
+<pinref part="U$44" gate="G$1" pin="GND@1"/>
 <wire x1="160.02" y1="25.4" x2="165.1" y2="25.4" width="0.1524" layer="91"/>
 <wire x1="165.1" y1="25.4" x2="165.1" y2="22.86" width="0.1524" layer="91"/>
@@
 <wire x1="172.72" y1="53.34" x2="175.26" y2="53.34" width="0.1524" layer="91"/>
 <wire x1="175.26" y1="53.34" x2="175.26" y2="17.78" width="0.1524" layer="91"/>
+<pinref part="U$44" gate="G$1" pin="FEED"/>
 <wire x1="175.26" y1="17.78" x2="160.02" y2="17.78" width="0.1524" layer="91"/>
 </segment>
