File: TBX01.sch (EAGLE design)
At the start: 75 parts, among them IC1 TPS62120, U3 STM32L151CCT6, U6 MCP73833, X2 FH12-10S-0.5SH, Y1 CRYSTAL.ABS07

Commit message: TBX01 v0.4
Parts:
- removed U$1: LS013B4DN04, sharp_LCD:LS013B4DN04
Changed lines of the file:
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@@
 <part name="JP1" library="SparkFun-Connectors" deviceset="USB" device="-MICROB"/>
 <part name="X2" library="con-hirose" deviceset="FH12-10S-0.5S" device="H"/>
-<part name="U$1" library="sharp_LCD" deviceset="LS013B4DN04" device=""/>
 <part name="U6" library="microbuilder" deviceset="MCP73833" device="" value="MCP73833"/>
 <part name="FRAME1" library="frames" deviceset="A3L-LOC" device=""/>
@@
 <instance part="X2" gate="-9" x="-124.46" y="-40.64" rot="R180"/>
 <instance part="X2" gate="-10" x="-124.46" y="-38.1" rot="R180"/>
-<instance part="U$1" gate="G$1" x="-182.88" y="-63.5"/>
 <instance part="U6" gate="G$1" x="-86.36" y="154.94"/>
 <instance part="FRAME1" gate="G$1" x="-200.66" y="-73.66"/>

Commit message: TBX01 v0.6
Parts:
- JP1: value USB-MICROB -> USB-RECEPTABLE-HIROSE-ZX62-AB-5PA(11); device SparkFun-Connectors:USB-MICROB -> daspilker:USB-RECEPTABLE-HIROSE-ZX62-AB-5PA(11)
Connections:
- net GND: now also U1-SLUG.TP
- net VIN: now also JP1.VCC; no longer JP1.VBUS
Changed lines of the file:
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@@
 <grid distance="0.1" unitdist="inch" unit="inch" style="lines" multiple="1" display="no" altdistance="0.01" altunitdist="inch" altunit="inch"/>
 <layers>
-<layer number="1" name="Top" color="4" fill="1" visible="no" active="no"/>
-<layer number="16" name="Bottom" color="1" fill="1" visible="no" active="no"/>
-<layer number="17" name="Pads" color="2" fill="1" visible="no" active="no"/>
-<layer number="18" name="Vias" color="2" fill="1" visible="no" active="no"/>
-<layer number="19" name="Unrouted" color="6" fill="1" visible="no" active="no"/>
-<layer number="20" name="Dimension" color="15" fill="1" visible="no" active="no"/>
-<layer number="21" name="tPlace" color="7" fill="1" visible="no" active="no"/>
-<layer number="22" name="bPlace" color="7" fill="1" visible="no" active="no"/>
-<layer number="23" name="tOrigins" color="15" fill="1" visible="no" active="no"/>
-<layer number="24" name="bOrigins" color="15" fill="1" visible="no" active="no"/>
-<layer number="25" name="tNames" color="7" fill="1" visible="no" active="no"/>
-<layer number="26" name="bNames" color="7" fill="1" visible="no" active="no"/>
-<layer number="27" name="tValues" color="7" fill="1" visible="no" active="no"/>
-<layer number="28" name="bValues" color="7" fill="1" visible="no" active="no"/>
+<layer number="1" name="Top" color="4" fill="1" visible="yes" active="no"/>
+<layer number="16" name="Bottom" color="1" fill="1" visible="yes" active="no"/>
+<layer number="17" name="Pads" color="2" fill="1" visible="yes" active="no"/>
+<layer number="18" name="Vias" color="2" fill="1" visible="yes" active="no"/>
+<layer number="19" name="Unrouted" color="6" fill="1" visible="yes" active="no"/>
+<layer number="20" name="Dimension" color="15" fill="1" visible="yes" active="no"/>
+<layer number="21" name="tPlace" color="7" fill="1" visible="yes" active="no"/>
+<layer number="22" name="bPlace" color="7" fill="1" visible="yes" active="no"/>
+<layer number="23" name="tOrigins" color="15" fill="1" visible="yes" active="no"/>
+<layer number="24" name="bOrigins" color="15" fill="1" visible="yes" active="no"/>
+<layer number="25" name="tNames" color="7" fill="1" visible="yes" active="no"/>
+<layer number="26" name="bNames" color="7" fill="1" visible="yes" active="no"/>
+<layer number="27" name="tValues" color="7" fill="1" visible="yes" active="no"/>
+<layer number="28" name="bValues" color="7" fill="1" visible="yes" active="no"/>
 <layer number="29" name="tStop" color="7" fill="3" visible="no" active="no"/>
 <layer number="30" name="bStop" color="7" fill="6" visible="no" active="no"/>
@@
 <layer number="35" name="tGlue" color="7" fill="4" visible="no" active="no"/>
 <layer number="36" name="bGlue" color="7" fill="5" visible="no" active="no"/>
-<layer number="37" name="tTest" color="7" fill="1" visible="no" active="no"/>
-<layer number="38" name="bTest" color="7" fill="1" visible="no" active="no"/>
+<layer number="37" name="tTest" color="7" fill="1" visible="yes" active="no"/>
+<layer number="38" name="bTest" color="7" fill="1" visible="yes" active="no"/>
 <layer number="39" name="tKeepout" color="4" fill="11" visible="no" active="no"/>
 <layer number="40" name="bKeepout" color="1" fill="11" visible="no" active="no"/>
@@
 <layer number="44" name="Drills" color="7" fill="1" visible="no" active="no"/>
 <layer number="45" name="Holes" color="7" fill="1" visible="no" active="no"/>
-<layer number="46" name="Milling" color="3" fill="1" visible="no" active="no"/>
-<layer number="47" name="Measures" color="7" fill="1" visible="no" active="no"/>
-<layer number="48" name="Document" color="7" fill="1" visible="no" active="no"/>
-<layer number="49" name="Reference" color="7" fill="1" visible="no" active="no"/>
-<layer number="50" name="dxf" color="7" fill="1" visible="no" active="no"/>
-<layer number="51" name="tDocu" color="7" fill="1" visible="no" active="no"/>
-<layer number="52" name="bDocu" color="7" fill="1" visible="no" active="no"/>
-<layer number="53" name="tGND_GNDA" color="7" fill="9" visible="no" active="no"/>
-<layer number="54" name="bGND_GNDA" color="1" fill="9" visible="no" active="no"/>
-<layer number="56" name="wert" color="7" fill="1" visible="no" active="no"/>
-<layer number="57" name="tCAD" color="7" fill="1" visible="no" active="no"/>
-<layer number="59" name="tCarbon" color="7" fill="1" visible="no" active="no"/>
-<layer number="60" name="bCarbon" color="7" fill="1" visible="no" active="no"/>
+<layer number="46" name="Milling" color="3" fill="1" visible="yes" active="no"/>
+<layer number="47" name="Measures" color="7" fill="1" visible="yes" active="no"/>
+<layer number="48" name="Document" color="7" fill="1" visible="yes" active="no"/>
+<layer number="49" name="Reference" color="7" fill="1" visible="yes" active="no"/>
+<layer number="50" name="dxf" color="7" fill="1" visible="yes" active="no"/>
+<layer number="51" name="tDocu" color="7" fill="1" visible="yes" active="no"/>
+<layer number="52" name="bDocu" color="7" fill="1" visible="yes" active="no"/>
+<layer number="53" name="tGND_GNDA" color="7" fill="9" visible="yes" active="no"/>
+<layer number="54" name="bGND_GNDA" color="1" fill="9" visible="yes" active="no"/>
+<layer number="56" name="wert" color="7" fill="1" visible="yes" active="no"/>
+<layer number="57" name="tCAD" color="7" fill="1" visible="yes" active="no"/>
+<layer number="59" name="tCarbon" color="7" fill="1" visible="yes" active="no"/>
+<layer number="60" name="bCarbon" color="7" fill="1" visible="yes" active="no"/>
 <layer number="90" name="Modules" color="5" fill="1" visible="yes" active="yes"/>
 <layer number="91" name="Nets" color="2" fill="1" visible="yes" active="yes"/>
@@
 </classes>
 <parts>
-<part name="JP1" library="SparkFun-Connectors" deviceset="USB" device="-MICROB"/>
 <part name="X2" library="con-hirose" deviceset="FH12-10S-0.5S" device="H"/>
 <part name="U6" library="microbuilder" deviceset="MCP73833" device="" value="MCP73833"/>
@@
 <part name="B6" library="alps" deviceset="SKSCLDE010" device=""/>
 <part name="B7" library="alps" deviceset="SKSCLDE010" device=""/>
+<part name="JP1" library="daspilker" deviceset="USB-RECEPTABLE" device="-HIROSE-ZX62-AB-5PA(11)"/>
+<part name="U$1" library="microbuilder" deviceset="GND" device=""/>
 </parts>
 <sheets>
@@
 </plain>
 <instances>
-<instance part="JP1" gate="G$1" x="-185.42" y="116.84" rot="R180"/>
 <instance part="X2" gate="-1" x="-124.46" y="-60.96" rot="R180"/>
 <instance part="X2" gate="-2" x="-124.46" y="-58.42" rot="R180"/>
@@
 <instance part="U$20" gate="G$1" x="-160.02" y="124.46"/>
 <instance part="U$24" gate="G$1" x="-139.7" y="175.26"/>
-<instance part="U$25" gate="G$1" x="-162.56" y="104.14"/>
+<instance part="U$25" gate="G$1" x="-162.56" y="96.52"/>
 <instance part="U$26" gate="G$1" x="-86.36" y="15.24"/>
 <instance part="C10" gate="G$1" x="-116.84" y="96.52"/>
@@
 <instance part="B6" gate="G$1" x="33.02" y="55.88"/>
 <instance part="B7" gate="G$1" x="137.16" y="134.62"/>
+<instance part="JP1" gate="G$1" x="-185.42" y="111.76" rot="R180"/>
+<instance part="U1" gate="-SLUG" x="167.64" y="106.68"/>
+<instance part="U$1" gate="G$1" x="167.64" y="88.9"/>
 </instances>
 <busses>
@@
 <net name="GND" class="0">
 <segment>
+<pinref part="U$25" gate="G$1" pin="GND"/>
+<wire x1="-162.56" y1="116.84" x2="-162.56" y2="99.06" width="0.1524" layer="91"/>
 <pinref part="JP1" gate="G$1" pin="GND"/>
-<wire x1="-182.88" y1="116.84" x2="-162.56" y2="116.84" width="0.1524" layer="91"/>
-<pinref part="U$25" gate="G$1" pin="GND"/>
-<wire x1="-162.56" y1="116.84" x2="-162.56" y2="106.68" width="0.1524" layer="91"/>
+<wire x1="-162.56" y1="116.84" x2="-177.8" y2="116.84" width="0.1524" layer="91"/>
 </segment>
 <segment>
@@
 <wire x1="73.66" y1="121.92" x2="73.66" y2="114.3" width="0.1524" layer="91"/>
 </segment>
+<segment>
+<pinref part="U1" gate="-SLUG" pin="TP"/>
+<pinref part="U$1" gate="G$1" pin="GND"/>
+<wire x1="167.64" y1="99.06" x2="167.64" y2="91.44" width="0.1524" layer="91"/>
+</segment>
 </net>
 <net name="VIN" class="0">
 <segment>
-<pinref part="JP1" gate="G$1" pin="VBUS"/>
-<wire x1="-182.88" y1="114.3" x2="-160.02" y2="114.3" width="0.1524" layer="91"/>
 <pinref part="U$20" gate="G$1" pin="VIN"/>
-<wire x1="-160.02" y1="114.3" x2="-160.02" y2="121.92" width="0.1524" layer="91"/>
+<wire x1="-160.02" y1="121.92" x2="-160.02" y2="106.68" width="0.1524" layer="91"/>
+<pinref part="JP1" gate="G$1" pin="VCC"/>
+<wire x1="-160.02" y1="106.68" x2="-177.8" y2="106.68" width="0.1524" layer="91"/>
 </segment>
 <segment>
@@
 <net name="D-" class="0">
 <segment>
+<label x="-167.64" y="111.76" size="1.778" layer="95"/>
+<pinref part="U3" gate="A" pin="PA11"/>
+<wire x1="-124.46" y1="109.22" x2="-124.46" y2="48.26" width="0.1524" layer="91"/>
+<wire x1="-124.46" y1="48.26" x2="-83.82" y2="48.26" width="0.1524" layer="91"/>
 <pinref part="JP1" gate="G$1" pin="D-"/>
-<label x="-167.64" y="111.76" size="1.778" layer="95"/>
-<wire x1="-182.88" y1="111.76" x2="-124.46" y2="111.76" width="0.1524" layer="91"/>
-<wire x1="-124.46" y1="111.76" x2="-124.46" y2="48.26" width="0.1524" layer="91"/>
-<pinref part="U3" gate="A" pin="PA11"/>
-<wire x1="-124.46" y1="48.26" x2="-83.82" y2="48.26" width="0.1524" layer="91"/>
+<wire x1="-177.8" y1="109.22" x2="-124.46" y2="109.22" width="0.1524" layer="91"/>
 </segment>
 </net>
 <net name="D+" class="0">
 <segment>
-<pinref part="JP1" gate="G$1" pin="D+"/>
 <label x="-167.64" y="109.22" size="1.778" layer="95"/>
 <pinref part="U3" gate="A" pin="PA12"/>
 <wire x1="-83.82" y1="45.72" x2="-127" y2="45.72" width="0.1524" layer="91"/>
-<wire x1="-127" y1="45.72" x2="-127" y2="109.22" width="0.1524" layer="91"/>
-<wire x1="-127" y1="109.22" x2="-182.88" y2="109.22" width="0.1524" layer="91"/>
+<wire x1="-127" y1="45.72" x2="-127" y2="111.76" width="0.1524" layer="91"/>
+<pinref part="JP1" gate="G$1" pin="D+"/>
+<wire x1="-127" y1="111.76" x2="-177.8" y2="111.76" width="0.1524" layer="91"/>
 </segment>
 </net>

Commit message: TBX01 v1.0
Parts:
- C1: value 1 uF -> 1uF
- C2, C3: value 4.7 uF -> 4.7uF
- C4: value 15 pF -> 15pF
- R1: value 14 kOhms -> 14k
- R2: value 4.7 kOhms -> 4.7k
- R3, R4, R7: value 4.7kOhms -> 4.7k
- R5: value 510 kOhms -> 510k
- R6: value 180 kOhms -> 180k
Changed lines of the file:
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@@
 <part name="FRAME1" library="frames" deviceset="A3L-LOC" device=""/>
 <part name="SUPPLY1" library="microbuilder" deviceset="GND" device=""/>
-<part name="C1" library="rcl" deviceset="C-EU" device="C0603" value="1 uF"/>
-<part name="C2" library="rcl" deviceset="C-EU" device="C0603" value="4.7 uF"/>
+<part name="C1" library="rcl" deviceset="C-EU" device="C0603" value="1uF"/>
+<part name="C2" library="rcl" deviceset="C-EU" device="C0603" value="4.7uF"/>
 <part name="SUPPLY5" library="microbuilder" deviceset="GND" device=""/>
 <part name="SUPPLY6" library="microbuilder" deviceset="GND" device=""/>
-<part name="R1" library="microbuilder" deviceset="RESISTOR" device="0603" value="14 kOhms"/>
+<part name="R1" library="microbuilder" deviceset="RESISTOR" device="0603" value="14k"/>
 <part name="SUPPLY8" library="microbuilder" deviceset="GND" device=""/>
-<part name="R2" library="microbuilder" deviceset="RESISTOR" device="0603" value="4.7 kOhms"/>
-<part name="R3" library="microbuilder" deviceset="RESISTOR" device="0603" value="4.7kOhms"/>
-<part name="R4" library="microbuilder" deviceset="RESISTOR" device="0603" value="4.7kOhms"/>
+<part name="R2" library="microbuilder" deviceset="RESISTOR" device="0603" value="4.7k"/>
+<part name="R3" library="microbuilder" deviceset="RESISTOR" device="0603" value="4.7k"/>
+<part name="R4" library="microbuilder" deviceset="RESISTOR" device="0603" value="4.7k"/>
 <part name="IC1" library="texas" deviceset="TPS62120" device=""/>
-<part name="C3" library="rcl" deviceset="C-EU" device="C0603" value="4.7 uF"/>
+<part name="C3" library="rcl" deviceset="C-EU" device="C0603" value="4.7uF"/>
 <part name="SUPPLY2" library="microbuilder" deviceset="GND" device=""/>
 <part name="L1" library="SparkFun-Passives" deviceset="INDUCTOR" device="1210" value="22uH"/>
 <part name="SUPPLY3" library="microbuilder" deviceset="GND" device=""/>
-<part name="C4" library="rcl" deviceset="C-EU" device="C0603" value="15 pF"/>
-<part name="R5" library="microbuilder" deviceset="RESISTOR" device="0603" value="510 kOhms"/>
-<part name="R6" library="microbuilder" deviceset="RESISTOR" device="0603" value="180 kOhms"/>
+<part name="C4" library="rcl" deviceset="C-EU" device="C0603" value="15pF"/>
+<part name="R5" library="microbuilder" deviceset="RESISTOR" device="0603" value="510k"/>
+<part name="R6" library="microbuilder" deviceset="RESISTOR" device="0603" value="180k"/>
 <part name="SUPPLY4" library="microbuilder" deviceset="GND" device=""/>
-<part name="R7" library="microbuilder" deviceset="RESISTOR" device="0603" value="4.7kOhms"/>
+<part name="R7" library="microbuilder" deviceset="RESISTOR" device="0603" value="4.7k"/>
 <part name="U3" library="ST Microelctronics_By_element14_Batch_1" deviceset="STM32L151CCT6" device=""/>
 <part name="U1" library="microbuilder" deviceset="NRF8001" device=""/>
@@
 <instance part="SUPPLY3" gate="G$1" x="25.4" y="139.7"/>
 <instance part="C4" gate="G$1" x="15.24" y="157.48" rot="R270"/>
-<instance part="R5" gate="G$1" x="5.08" y="160.02"/>
-<instance part="R6" gate="G$1" x="5.08" y="154.94"/>
+<instance part="R5" gate="G$1" x="5.08" y="160.02" smashed="yes">
+<attribute name="NAME" x="2.54" y="162.052" size="1.27" layer="95" font="vector"/>
+<attribute name="VALUE" x="10.16" y="159.385" size="1.27" layer="96" font="vector"/>
+</instance>
+<instance part="R6" gate="G$1" x="5.08" y="154.94" smashed="yes">
+<attribute name="NAME" x="2.54" y="156.972" size="1.27" layer="95" font="vector"/>
+<attribute name="VALUE" x="-5.08" y="154.305" size="1.27" layer="96" font="vector"/>
+</instance>
 <instance part="SUPPLY4" gate="G$1" x="20.32" y="139.7"/>
 <instance part="R7" gate="G$1" x="30.48" y="149.86" rot="R90"/>
@@
 <instance part="U$25" gate="G$1" x="-162.56" y="96.52"/>
 <instance part="U$26" gate="G$1" x="-86.36" y="15.24"/>
-<instance part="C10" gate="G$1" x="-116.84" y="96.52"/>
-<instance part="C11" gate="G$1" x="-106.68" y="99.06" rot="R180"/>
-<instance part="C12" gate="G$1" x="-96.52" y="96.52"/>
+<instance part="C10" gate="G$1" x="-116.84" y="96.52" smashed="yes">
+<attribute name="NAME" x="-119.38" y="101.6" size="1.27" layer="95" font="vector"/>
+<attribute name="VALUE" x="-119.38" y="93.98" size="1.27" layer="96" font="vector"/>
+</instance>
+<instance part="C11" gate="G$1" x="-106.68" y="99.06" smashed="yes" rot="R180">
+<attribute name="NAME" x="-106.68" y="101.6" size="1.27" layer="95" font="vector" rot="R180"/>
+<attribute name="VALUE" x="-104.14" y="96.52" size="1.27" layer="96" font="vector" rot="R180"/>
+</instance>
+<instance part="C12" gate="G$1" x="-96.52" y="96.52" smashed="yes">
+<attribute name="NAME" x="-93.98" y="99.06" size="1.27" layer="95" font="vector"/>
+<attribute name="VALUE" x="-93.98" y="96.52" size="1.27" layer="96" font="vector"/>
+</instance>
 <instance part="U$27" gate="G$1" x="-106.68" y="109.22"/>
 <instance part="U$29" gate="G$1" x="-106.68" y="86.36"/>

Commit message: TBX01 v1.0-r201510201242
Changed lines of the file:
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@@
 <drawing>
 <settings>
-<setting alwaysvectorfont="no"/>
+<setting alwaysvectorfont="yes"/>
 <setting verticaltext="up"/>
 </settings>
 <grid distance="0.1" unitdist="inch" unit="inch" style="lines" multiple="1" display="no" altdistance="0.01" altunitdist="inch" altunit="inch"/>
 <layers>
-<layer number="1" name="Top" color="4" fill="1" visible="yes" active="no"/>
-<layer number="16" name="Bottom" color="1" fill="1" visible="yes" active="no"/>
-<layer number="17" name="Pads" color="2" fill="1" visible="yes" active="no"/>
-<layer number="18" name="Vias" color="2" fill="1" visible="yes" active="no"/>
-<layer number="19" name="Unrouted" color="6" fill="1" visible="yes" active="no"/>
-<layer number="20" name="Dimension" color="15" fill="1" visible="yes" active="no"/>
-<layer number="21" name="tPlace" color="7" fill="1" visible="yes" active="no"/>
-<layer number="22" name="bPlace" color="7" fill="1" visible="yes" active="no"/>
-<layer number="23" name="tOrigins" color="15" fill="1" visible="yes" active="no"/>
-<layer number="24" name="bOrigins" color="15" fill="1" visible="yes" active="no"/>
-<layer number="25" name="tNames" color="7" fill="1" visible="yes" active="no"/>
-<layer number="26" name="bNames" color="7" fill="1" visible="yes" active="no"/>
-<layer number="27" name="tValues" color="7" fill="1" visible="yes" active="no"/>
-<layer number="28" name="bValues" color="7" fill="1" visible="yes" active="no"/>
+<layer number="1" name="Top" color="4" fill="1" visible="no" active="no"/>
+<layer number="16" name="Bottom" color="1" fill="1" visible="no" active="no"/>
+<layer number="17" name="Pads" color="2" fill="1" visible="no" active="no"/>
+<layer number="18" name="Vias" color="2" fill="1" visible="no" active="no"/>
+<layer number="19" name="Unrouted" color="6" fill="1" visible="no" active="no"/>
+<layer number="20" name="Dimension" color="15" fill="1" visible="no" active="no"/>
+<layer number="21" name="tPlace" color="7" fill="1" visible="no" active="no"/>
+<layer number="22" name="bPlace" color="7" fill="1" visible="no" active="no"/>
+<layer number="23" name="tOrigins" color="15" fill="1" visible="no" active="no"/>
+<layer number="24" name="bOrigins" color="15" fill="1" visible="no" active="no"/>
+<layer number="25" name="tNames" color="7" fill="1" visible="no" active="no"/>
+<layer number="26" name="bNames" color="7" fill="1" visible="no" active="no"/>
+<layer number="27" name="tValues" color="7" fill="1" visible="no" active="no"/>
+<layer number="28" name="bValues" color="7" fill="1" visible="no" active="no"/>
 <layer number="29" name="tStop" color="7" fill="3" visible="no" active="no"/>
 <layer number="30" name="bStop" color="7" fill="6" visible="no" active="no"/>
@@
 <layer number="35" name="tGlue" color="7" fill="4" visible="no" active="no"/>
 <layer number="36" name="bGlue" color="7" fill="5" visible="no" active="no"/>
-<layer number="37" name="tTest" color="7" fill="1" visible="yes" active="no"/>
-<layer number="38" name="bTest" color="7" fill="1" visible="yes" active="no"/>
+<layer number="37" name="tTest" color="7" fill="1" visible="no" active="no"/>
+<layer number="38" name="bTest" color="7" fill="1" visible="no" active="no"/>
 <layer number="39" name="tKeepout" color="4" fill="11" visible="no" active="no"/>
 <layer number="40" name="bKeepout" color="1" fill="11" visible="no" active="no"/>
@@
 <layer number="44" name="Drills" color="7" fill="1" visible="no" active="no"/>
 <layer number="45" name="Holes" color="7" fill="1" visible="no" active="no"/>
-<layer number="46" name="Milling" color="3" fill="1" visible="yes" active="no"/>
-<layer number="47" name="Measures" color="7" fill="1" visible="yes" active="no"/>
-<layer number="48" name="Document" color="7" fill="1" visible="yes" active="no"/>
-<layer number="49" name="Reference" color="7" fill="1" visible="yes" active="no"/>
-<layer number="50" name="dxf" color="7" fill="1" visible="yes" active="no"/>
-<layer number="51" name="tDocu" color="7" fill="1" visible="yes" active="no"/>
-<layer number="52" name="bDocu" color="7" fill="1" visible="yes" active="no"/>
-<layer number="53" name="tGND_GNDA" color="7" fill="9" visible="yes" active="no"/>
-<layer number="54" name="bGND_GNDA" color="1" fill="9" visible="yes" active="no"/>
-<layer number="56" name="wert" color="7" fill="1" visible="yes" active="no"/>
-<layer number="57" name="tCAD" color="7" fill="1" visible="yes" active="no"/>
-<layer number="59" name="tCarbon" color="7" fill="1" visible="yes" active="no"/>
-<layer number="60" name="bCarbon" color="7" fill="1" visible="yes" active="no"/>
+<layer number="46" name="Milling" color="3" fill="1" visible="no" active="no"/>
+<layer number="47" name="Measures" color="7" fill="1" visible="no" active="no"/>
+<layer number="48" name="Document" color="7" fill="1" visible="no" active="no"/>
+<layer number="49" name="Reference" color="7" fill="1" visible="no" active="no"/>
+<layer number="50" name="dxf" color="7" fill="1" visible="no" active="no"/>
+<layer number="51" name="tDocu" color="7" fill="1" visible="no" active="no"/>
+<layer number="52" name="bDocu" color="7" fill="1" visible="no" active="no"/>
+<layer number="53" name="tGND_GNDA" color="7" fill="9" visible="no" active="no"/>
+<layer number="54" name="bGND_GNDA" color="1" fill="9" visible="no" active="no"/>
+<layer number="56" name="wert" color="7" fill="1" visible="no" active="no"/>
+<layer number="57" name="tCAD" color="7" fill="1" visible="no" active="no"/>
+<layer number="59" name="tCarbon" color="7" fill="1" visible="no" active="no"/>
+<layer number="60" name="bCarbon" color="7" fill="1" visible="no" active="no"/>
 <layer number="90" name="Modules" color="5" fill="1" visible="yes" active="yes"/>
 <layer number="91" name="Nets" color="2" fill="1" visible="yes" active="yes"/>
@@
 <instance part="B6" gate="G$1" x="33.02" y="55.88"/>
 <instance part="B7" gate="G$1" x="137.16" y="134.62"/>
-<instance part="JP1" gate="G$1" x="-185.42" y="111.76" rot="R180"/>
+<instance part="JP1" gate="G$1" x="-185.42" y="111.76" smashed="yes" rot="R180">
+<attribute name="NAME" x="-180.594" y="103.632" size="1.778" layer="95" rot="R180"/>
+<attribute name="VALUE" x="-137.16" y="121.666" size="1.778" layer="96" rot="R180"/>
+</instance>
 <instance part="U1" gate="-SLUG" x="167.64" y="106.68"/>
 <instance part="U$1" gate="G$1" x="167.64" y="88.9"/>
